File: TANDY_200_Dual_RAM_tsop.kicad_sch (KiCad schematic)
At the start: 5 parts, among them J1 Conn_01x01_Male, J2 TANDY_26-3688, U1 628128_TSOP32, U2 74LVC1G08

Commit message: ground paths, footprints, sch symbols
Other:
- title: TANDY 200 Dual RAM (tsop) -> TANDY 200 Dual RAM tsop
Changed lines of the file:
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@@
   (paper "USLetter")
   (title_block
-    (title "TANDY 200 Dual RAM (tsop)")
-    (date "2022-09-16")
+    (title "TANDY 200 Dual RAM tsop")
+    (date "2022-09-22")
     (rev "001")
     (company "b.kenyon.w@gmail.com")
@@
       (effects (font (size 1.27 1.27)) hide)
     )
-    (property "Value" "VCC" (id 1) (at 76.2 74.422 0))
+    (property "Value" "VCC" (id 1) (at 76.2 74.93 0))
     (property "Footprint" "" (id 2) (at 76.2 78.74 0)
       (effects (font (size 1.27 1.27)) hide)
@@
       (effects (font (size 1.27 1.27)) hide)
     )
-    (property "Value" "GND" (id 1) (at 76.2 129.032 90))
+    (property "Value" "GND" (id 1) (at 76.2 128.27 0))
     (property "Footprint" "" (id 2) (at 76.2 124.46 0)
       (effects (font (size 1.27 1.27)) hide)
@@
       (effects (font (size 1.27 1.27)) hide)
     )
-    (property "Value" "VCC" (id 1) (at 165.1 61.722 0))
+    (property "Value" "VCC" (id 1) (at 165.1 62.23 0))
     (property "Footprint" "" (id 2) (at 165.1 66.04 0)
       (effects (font (size 1.27 1.27)) hide)
@@
       (effects (font (size 1.27 1.27)) hide)
     )
-    (property "Value" "GND" (id 1) (at 165.1 75.692 90))
+    (property "Value" "GND" (id 1) (at 165.1 74.93 0))
     (property "Footprint" "" (id 2) (at 165.1 71.12 0)
       (effects (font (size 1.27 1.27)) hide)
@@
   )
   (symbol (lib_id "000_LOCAL:74LVC1G08") (at 133.35 113.03 0) (unit 1)
-    (in_bom yes) (on_board yes) (fields_autoplaced)
-    (property "Reference" "U2" (id 0) (at 132.715 105.41 0))
-    (property "Value" "74LVC1G08" (id 1) (at 132.715 107.95 0))
+    (in_bom yes) (on_board yes)
+    (property "Reference" "U2" (id 0) (at 133.35 109.22 0))
+    (property "Value" "74LVC1G08" (id 1) (at 133.35 116.84 0))
     (property "Footprint" "000_LOCAL:SOT-23-5" (id 2) (at 133.35 113.03 0)
       (effects (font (size 1.27 1.27)) hide)
@@
     (pin "2")
   )
+  (symbol (lib_id "power:VCC") (at 190.5 78.74 0) (unit 1)
+    (in_bom yes) (on_board yes)
+    (property "Reference" "#PWR0103" (id 0) (at 190.5 82.55 0)
+      (effects (font (size 1.27 1.27)) hide)
+    )
+    (property "Value" "VCC" (id 1) (at 190.5 74.93 0))
+    (property "Footprint" "" (id 2) (at 190.5 78.74 0)
+      (effects (font (size 1.27 1.27)) hide)
+    )
+    (property "Datasheet" "" (id 3) (at 190.5 78.74 0)
+      (effects (font (size 1.27 1.27)) hide)
+    )
+    (pin "1")
+  )
+  (symbol (lib_id "power:GND") (at 190.5 129.54 0) (unit 1)
+    (in_bom yes) (on_board yes)
+    (property "Reference" "#PWR0101" (id 0) (at 190.5 135.89 0)
+      (effects (font (size 1.27 1.27)) hide)
+    )
+    (property "Value" "GND" (id 1) (at 190.5 133.35 0))
+    (property "Footprint" "" (id 2) (at 190.5 129.54 0)
+      (effects (font (size 1.27 1.27)) hide)
+    )
+    (property "Datasheet" "" (id 3) (at 190.5 129.54 0)
+      (effects (font (size 1.27 1.27)) hide)
+    )
+    (pin "1")
+  )
   (symbol (lib_id "000_LOCAL:628128_TSOP32") (at 190.5 104.14 0) (unit 1)
     (in_bom yes) (on_board yes)
@@
       (effects (font (size 1.27 1.27)) (justify left bottom))
     )
-    (property "Value" "628128_TSOP32" (id 1) (at 191.77 80.01 0)
+    (property "Value" "628128_TSOP32" (id 1) (at 192.024 80.264 0)
       (effects (font (size 1.27 1.27)) (justify left bottom))
     )
@@
   )
   (symbol_instances
+    (path "/a14f88dd-772e-4609-8a0c-993194aa9d54"
+      (reference "#PWR0101") (unit 1) (value "GND") (footprint "")
+    )
     (path "/009aec29-5876-4a82-9c35-f7f614fcec3b"
       (reference "#PWR0102") (unit 1) (value "GND") (footprint "")
     )
+    (path "/899f2574-716b-46ca-8e79-8c6668cbc95d"
+      (reference "#PWR0103") (unit 1) (value "VCC") (footprint "")
+    )
     (path "/00000000-0000-0000-0000-000060782b2b"
